File: electronics/PCB/S77_Eggbot.sch (EAGLE design)
At the start: 5 parts, among them U1 CR_LM2596, U2 S2_MINI, U3 CARRIER_A4988, U4 CARRIER_A4988, X1 POLLIN_JACK_A

Commit message: WIP: fix board dimension and place components
Parts:
- added C1, C2: 100µF/35V/0R056, rcl:CPOL-EUE3.5-8
- added D1: 1N5822, lib_s77_eggbot:1N5822
- added JP1, JP2, JP3: (no value), pinhead:PINHD-1X4
- added JP4: (no value), pinhead:PINHD-1X8
- added SERVO: (no value), pinhead:PINHD-1X3
- added SJ1, SJ2, SJ3, SJ4, SJ5, SJ6: (no value), jumper:SJ
- added X2, X3: B6B-PH, lib_s77_eggbot:B6B-PH
- X1: value POLLIN_JACK_A -> PWR
Connections:
- new net +3V3: JP1.3, SJ1.1, SJ2.1, SJ3.1, SJ4.1, SJ5.1, SJ6.1, U2.+3V3, U3.!RESET, U3.!SLEEP, U3.VDD, U4.!RESET, U4.!SLEEP
- new net +5V: JP1.2, U1.OUT
- new net N$10: JP3.4, U4.OUT_2B, X3-6.1
- new net N$11: SJ1.2, U3.MS1
- new net N$12: SJ2.2, U3.MS2
- new net N$13: SJ3.2, U3.MS3
- new net N$14: U3.!ENABLE
- new net N$15: U3.DIR
- new net N$16: U3.STEP
- new net N$17: SJ4.2, U4.MS1
- new net N$18: SJ5.2, U4.MS2
- new net N$19: SJ6.2, U4.MS3
- new net N$2: JP2.1, U3.OUT_1B, X2-1.1
- new net N$3: D1.A, X1.1
- new net N$4: JP2.2, U3.OUT_1A, X2-2.1
- new net N$5: JP2.3, U3.OUT_2A, X2-4.1
- new net N$6: JP2.4, U3.OUT_2B, X2-6.1
- new net N$7: JP3.1, U4.OUT_1B, X3-1.1
- new net N$8: JP3.2, U4.OUT_1A, X3-2.1
- new net N$9: JP3.3, U4.OUT_2A, X3-4.1
- new net VMOT: C1.+, C2.+, D1.C, JP1.1, U1.IN, U3.VMOT, U4.VMOT
- net GND: now also C1.-, C2.-, JP1.4, X1.2
Other:
- note added: "12V TODO: Bereich spezifizieren?"
- note added: "2x Pollin 94-310690 MINEBEA Schrittmotor 17PM-K374BN01CN"
- note added: "40V/3A"
- note added: "BLU (B) - ORG (/B) RED (A) - YEL (/A)"
- note added: "Braun - GND Rot - 5V Orange - PWM"
- note added: "MS1 + MS3 100k, MS2 50k internal pull-down"
- moved on the sheet: U1, U2, U3, U4, X1

Commit message: first version of schematic and layout
Parts:
- JP4: device pinhead:PINHD-1X8 -> pinhead:PINHD-1X12
Connections:
- removed net N$1: U1.GND@1, U1.GND@2
- removed net N$14: U3.!ENABLE
- removed net N$15: U3.DIR
- removed net N$16: U3.STEP
- new net DIR1: U2.IO2, U3.DIR
- new net DIR2: U2.IO4, U4.DIR
- new net N$20: JP4.4, U2.IO7/SCK
- new net N$21: JP4.3, U2.IO9/MISO
- new net N$22: JP4.2, U2.IO11/MOSI
- new net N$23: JP4.5, U2.IO17
- new net N$24: JP4.6, U2.IO18/PU10K
- new net N$25: JP4.7, U2.IO33/SDA
- new net N$26: JP4.9, U2.IO34
- new net N$27: JP4.8, U2.IO35/SCL
- new net N$28: JP4.11, U2.IO36
- new net N$29: JP4.10, U2.IO37
- new net SERVO_PWM: SERVO.3, U2.IO6
- new net STEP1: U2.IO3, U3.STEP
- new net STEP2: U2.IO5, U4.STEP
- new net STEPPER_EN: U2.IO1, U3.!ENABLE, U4.!ENABLE
- net +3V3: now also JP4.1, U4.VDD
- net +5V: now also SERVO.2, U2.VBUS
- net GND: now also JP4.12, SERVO.1, U1.GND@1, U1.GND@2
- net N$4: now also X2-3.1; no longer X2-2.1
- net N$8: now also X3-3.1; no longer X3-2.1

Commit message: PCB: fix smaller details, update docs
Other:
- note added: "Achtung: Ausgangsspannung am Trimmer auf 5V einstellen, bevor die anderen Module gesteckt werden!"
- note added: "EN has internal 10k pull-up to +3V3"
- note added: "Graupner/JR Belegung:"
- note added: "IOs, DAC, SPI, I2C for external use"
- note added: "Input 9V - 30V"
- note added: "for external use"
- note added: "https://github.com/section77/eggbot77 by andy, 25.01.2024"
- note removed: "12V TODO: Bereich spezifizieren?"
- note removed: "Achtung: Ausgangsspannung auf 5V einstellen, bevor die anderen Module gesteckt werden!"
- moved on the sheet: SERVO
Changed lines of the file:
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@@
 <sheet>
 <plain>
-<text x="58.42" y="160.02" size="1.778" layer="97">Achtung:
-Ausgangsspannung auf 5V
-einstellen, bevor die anderen
+<text x="50.8" y="162.56" size="1.778" layer="97">Achtung:
+Ausgangsspannung am Trimmer
+auf 5V einstellen, bevor die anderen
 Module gesteckt werden!</text>
-<text x="7.62" y="162.56" size="1.9304" layer="97">12V
-TODO: Bereich spezifizieren?</text>
+<text x="7.62" y="162.56" size="1.9304" layer="97">Input
+9V - 30V</text>
 <text x="30.988" y="146.558" size="1.778" layer="96">40V/3A</text>
 <text x="251.46" y="88.9" size="1.778" layer="96" rot="R90">2x Pollin 94-310690
@@
 YEL (/A)
  </text>
-<text x="91.44" y="17.78" size="1.6764" layer="96" align="center-left">Braun - GND
+<text x="86.36" y="15.24" size="1.6764" layer="96" align="center-left">Braun - GND
 Rot - 5V
 Orange - PWM</text>
@@
 YEL (/A)
  </text>
+<text x="101.6" y="160.02" size="1.9304" layer="97">for external use</text>
+<text x="114.3" y="33.02" size="1.9304" layer="97" rot="R90">IOs, DAC, SPI, I2C for external use</text>
+<text x="22.86" y="86.36" size="1.778" layer="97">EN has internal
+10k pull-up to +3V3</text>
+<text x="165.1" y="15.24" size="1.9304" layer="94">https://github.com/section77/eggbot77
+by andy, 25.01.2024</text>
+<text x="86.36" y="22.86" size="1.6764" layer="96" align="center-left">Graupner/JR
+Belegung:</text>
 </plain>
 <instances>
@@
 <instance part="X2" gate="-5" x="233.68" y="132.08"/>
 <instance part="X2" gate="-6" x="233.68" y="129.54"/>
-<instance part="SERVO" gate="A" x="88.9" y="17.78"/>
+<instance part="SERVO" gate="A" x="81.28" y="15.24"/>
 <instance part="SJ1" gate="1" x="162.56" y="132.08" smashed="yes">
 <attribute name="VALUE" x="160.02" y="128.27" size="1.778" layer="96"/>
@@
 <segment>
 <pinref part="SERVO" gate="A" pin="1"/>
-<wire x1="86.36" y1="20.32" x2="76.2" y2="20.32" width="0.1524" layer="91"/>
-<label x="76.2" y="20.32" size="1.27" layer="95" rot="R180" xref="yes"/>
+<wire x1="78.74" y1="17.78" x2="68.58" y2="17.78" width="0.1524" layer="91"/>
+<label x="68.58" y="17.78" size="1.27" layer="95" rot="R180" xref="yes"/>
 </segment>
 <segment>
@@
 <segment>
 <pinref part="SERVO" gate="A" pin="2"/>
-<wire x1="86.36" y1="17.78" x2="76.2" y2="17.78" width="0.1524" layer="91"/>
-<label x="76.2" y="17.78" size="1.27" layer="95" rot="R180" xref="yes"/>
+<wire x1="78.74" y1="15.24" x2="68.58" y2="15.24" width="0.1524" layer="91"/>
+<label x="68.58" y="15.24" size="1.27" layer="95" rot="R180" xref="yes"/>
 </segment>
 <segment>
@@
 <segment>
 <pinref part="SERVO" gate="A" pin="3"/>
-<wire x1="86.36" y1="15.24" x2="76.2" y2="15.24" width="0.1524" layer="91"/>
-<label x="76.2" y="15.24" size="1.27" layer="95" rot="R180" xref="yes"/>
-</segment>
-</net>
+<wire x1="78.74" y1="12.7" x2="68.58" y2="12.7" width="0.1524" layer="91"/>
+<label x="68.58" y="12.7" size="1.27" layer="95" rot="R180" xref="yes"/>
+</segment>
+</net>

Commit message: PCB: update date
Other:
- note added: "ATTENTION: 3,3V PWM voltage level Some servos might have problems FIXME: consider level shifter"
- note added: "Graupner/JR:"
- note added: "https://github.com/section77/eggbot77 by andy, 09.02.2024"
- note removed: "Graupner/JR Belegung:"
- note removed: "https://github.com/section77/eggbot77 by andy, 25.01.2024"
Changed lines of the file:
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@@
 10k pull-up to +3V3</text>
 <text x="165.1" y="15.24" size="1.9304" layer="94">https://github.com/section77/eggbot77
-by andy, 25.01.2024</text>
-<text x="86.36" y="22.86" size="1.6764" layer="96" align="center-left">Graupner/JR
-Belegung:</text>
+by andy, 09.02.2024</text>
+<text x="86.36" y="22.86" size="1.6764" layer="96" align="center-left">Graupner/JR:</text>
+<text x="104.14" y="10.16" size="1.9304" layer="97">ATTENTION:
+3,3V PWM voltage level
+Some servos might have problems
+FIXME: consider level shifter</text>
 </plain>
 <instances>
