File: electronics/PCB/S77_Eggbot.brd (EAGLE design)
At the start: 70 x 70 mm, 21 parts, among them U1 CR_LM2596, U2 S2_MINI, U3 CARRIER_A4988, U4 CARRIER_A4988, X1 PWR, X2 B6B-PH, X3 B6B-PH

Commit message: PCB: added 3.3V<->5V levelshifter for servo PWM, update exports
Parts:
- added Q1: BSS138, bss138_10:SOT23
- added R1, R2: 4k7, rcl:R1206
- added SJ7: n.o., jumper:SJ
Connections:
- new net N$1: Q1.3, R1.1, SERVO.3, SJ7.2
- net +3V3: now also Q1.1, R2.2
- net +5V: now also R1.2
- net SERVO_PWM: now also Q1.2, R2.1, SJ7.1; no longer SERVO.3
Routing:
- net N$1: track 0.00 -> 39.5 mm
- net +3V3: track 191.0 -> 219.6 mm, vias 1 -> 2
- net SERVO_PWM: track 47.4 -> 19.1 mm
- net +5V: track 141.7 -> 150.7 mm
Other:
- board text added: "eggbot77 section77.de 12.02.2024"
- board text removed: "eggbot77 section77.de 09.02.2024"
Changed lines of the file:
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@@
 <setting verticaltext="up"/>
 </settings>
-<grid distance="0.05" unitdist="mm" unit="mm" style="lines" multiple="1" display="yes" altdistance="0.025" altunitdist="inch" altunit="inch"/>
+<grid distance="0.5" unitdist="mm" unit="mm" style="lines" multiple="1" display="yes" altdistance="0.025" altunitdist="inch" altunit="inch"/>
 <layers>
-<layer number="1" name="Top" color="4" fill="1" visible="no" active="yes"/>
+<layer number="1" name="Top" color="4" fill="1" visible="yes" active="yes"/>
 <layer number="2" name="Route2" color="1" fill="3" visible="no" active="no"/>
 <layer number="3" name="Route3" color="4" fill="3" visible="no" active="no"/>
@@
 <layer number="19" name="Unrouted" color="6" fill="1" visible="yes" active="yes"/>
 <layer number="20" name="Dimension" color="15" fill="1" visible="yes" active="yes"/>
-<layer number="21" name="tPlace" color="7" fill="1" visible="no" active="yes"/>
+<layer number="21" name="tPlace" color="7" fill="1" visible="yes" active="yes"/>
 <layer number="22" name="bPlace" color="7" fill="1" visible="yes" active="yes"/>
-<layer number="23" name="tOrigins" color="15" fill="1" visible="no" active="yes"/>
+<layer number="23" name="tOrigins" color="15" fill="1" visible="yes" active="yes"/>
 <layer number="24" name="bOrigins" color="15" fill="1" visible="yes" active="yes"/>
-<layer number="25" name="tNames" color="7" fill="1" visible="no" active="yes"/>
+<layer number="25" name="tNames" color="7" fill="1" visible="yes" active="yes"/>
 <layer number="26" name="bNames" color="7" fill="1" visible="yes" active="yes"/>
 <layer number="27" name="tValues" color="7" fill="1" visible="yes" active="yes"/>
@@
 <wire x1="70" y1="70" x2="0" y2="70" width="0" layer="20"/>
 <wire x1="0" y1="70" x2="0" y2="0" width="0" layer="20"/>
-<text x="53.715" y="5.285" size="1.4224" layer="21" font="vector" rot="R180" align="center-left">PWM
+<text x="54.215" y="5.485" size="1.4224" layer="21" font="vector" rot="R180" align="center-left">PWM
 +5V
 GND</text>
@@
 <text x="26.73" y="40.98" size="2.54" layer="26" font="vector" rot="MR180" align="center">eggbot77
 section77.de
-09.02.2024</text>
+12.02.2024</text>
 <text x="39.215" y="41.285" size="1.4224" layer="21" font="vector" rot="R180" align="center-left">ATTENTION:
 Trim output to
@@
 <attribute name="VALUE" x="13.76" y="1.325" size="1.27" layer="27"/>
 </element>
+<element name="Q1" library="bss138_10" package="SOT23" value="BSS138" x="29.5" y="20" smashed="yes" rot="R180">
+<attribute name="OC_FARNELL" value="9845330" x="29.5" y="20" size="1.778" layer="27" rot="R180" display="off"/>
+<attribute name="MPN" value="BSS138" x="29.5" y="20" size="1.778" layer="27" rot="R180" display="off"/>
+<attribute name="OC_NEWARK" value="67R2009" x="29.5" y="20" size="1.778" layer="27" rot="R180" display="off"/>
+<attribute name="MF" value="Fairchild" x="29.5" y="20" size="1.778" layer="27" rot="R180" display="off"/>
+<attribute name="NAME" x="31.4" y="19.35" size="1.27" layer="25"/>
+</element>
+<element name="R1" library="rcl" package="R1206" value="4k7" x="47.5" y="7" smashed="yes" rot="R270">
+<attribute name="NAME" x="47.5" y="4" size="1.27" layer="25" rot="R270" align="center-left"/>
+<attribute name="VALUE" x="44.96" y="8.27" size="1.27" layer="27" rot="R270"/>
+</element>
+<element name="SJ7" library="jumper" package="SJ" value="n.o." x="24.5" y="23" smashed="yes" rot="R270">
+<attribute name="NAME" x="24.5" y="25.5" size="1.27" layer="25" ratio="10" align="bottom-center"/>
+<attribute name="VALUE" x="24.5" y="22.5999" size="0.02" layer="27" rot="R270"/>
+</element>
+<element name="R2" library="rcl" package="R1206" value="4k7" x="29.7" y="25.75" smashed="yes">
+<attribute name="NAME" x="28.43" y="27.02" size="1.27" layer="25"/>
+<attribute name="VALUE" x="28.43" y="23.21" size="1.27" layer="27"/>
+</element>
 </elements>
 <signals>
@@
 <wire x1="51" y1="1.5" x2="55" y2="5.5" width="1.27" layer="16"/>
 <wire x1="55" y1="5.5" x2="56.5" y2="5.5" width="1.27" layer="16"/>
+<contactref element="R1" pad="2"/>
+<wire x1="47.5" y1="5.578" x2="47.578" y2="5.5" width="0.6096" layer="1"/>
+<wire x1="47.578" y1="5.5" x2="56.5" y2="5.5" width="0.6096" layer="1"/>
 </signal>
 <signal name="GND1">
@@
 <wire x1="54.08" y1="14.92" x2="51.5" y2="17.5" width="1.27" layer="16"/>
 <wire x1="51.5" y1="17.5" x2="51.5" y2="20" width="1.27" layer="16"/>
-<wire x1="51.5" y1="20" x2="51.5" y2="42.5" width="1.27" layer="16"/>
+<wire x1="51.5" y1="20" x2="51.5" y2="33.5" width="1.27" layer="16"/>
+<wire x1="51.5" y1="33.5" x2="51.5" y2="42.5" width="1.27" layer="16"/>
 <wire x1="51.5" y1="42.5" x2="51.5" y2="57.5" width="1.27" layer="16"/>
 <wire x1="51.5" y1="57.5" x2="49" y2="60" width="1.27" layer="16"/>
@@
 <wire x1="8.89" y1="33.73" x2="6.35" y2="31.19" width="0.4064" layer="16"/>
 <wire x1="6.35" y1="31.19" x2="6.35" y2="21.59" width="0.4064" layer="16"/>
+<contactref element="R2" pad="2"/>
+<contactref element="Q1" pad="1"/>
+<wire x1="30.45" y1="21" x2="31.122" y2="21.672" width="0.6096" layer="1"/>
+<wire x1="31.122" y1="21.672" x2="31.122" y2="25.75" width="0.6096" layer="1"/>
+<wire x1="31.122" y1="25.75" x2="32.25" y2="25.75" width="0.6096" layer="1"/>
+<wire x1="32.25" y1="25.75" x2="40" y2="33.5" width="0.6096" layer="1"/>
+<wire x1="40" y1="33.5" x2="51.5" y2="33.5" width="0.6096" layer="1"/>
+<via x="51.5" y="33.5" extent="1-16" drill="0.8" diameter="1.27" shape="octagon"/>
 </signal>
 <signal name="N$11">
@@
 <signal name="SERVO_PWM">
 <contactref element="U2" pad="20"/>
-<contactref element="SERVO" pad="3"/>
-<wire x1="19.05" y1="31.19" x2="19.05" y2="30.6" width="0.6096" layer="16"/>
-<wire x1="19.05" y1="30.6" x2="39.65" y2="10" width="0.6096" layer="16"/>
-<wire x1="39.65" y1="10" x2="54.54" y2="10" width="0.6096" layer="16"/>
-<wire x1="56.5" y1="8.04" x2="54.54" y2="10" width="0.6096" layer="16"/>
+<contactref element="Q1" pad="2"/>
+<contactref element="R2" pad="1"/>
+<contactref element="SJ7" pad="1"/>
+<wire x1="28.55" y1="21" x2="28.278" y2="21.272" width="0.6096" layer="1"/>
+<wire x1="28.278" y1="21.272" x2="28.278" y2="25.75" width="0.6096" layer="1"/>
+<wire x1="28.278" y1="25.75" x2="26.488" y2="25.75" width="0.6096" layer="1"/>
+<wire x1="26.488" y1="25.75" x2="24.5" y2="23.762" width="0.6096" layer="1"/>
+<wire x1="19.05" y1="31.19" x2="19.05" y2="29.212" width="0.6096" layer="1"/>
+<wire x1="19.05" y1="29.212" x2="24.5" y2="23.762" width="0.6096" layer="1"/>
 </signal>
 <signal name="N$20">
@@
 <wire x1="26.11" y1="8.89" x2="24.13" y2="10.87" width="0.4064" layer="16"/>
 </signal>
+<signal name="N$1">
+<contactref element="Q1" pad="3"/>
+<contactref element="R1" pad="1"/>
+<contactref element="SERVO" pad="3"/>
+<contactref element="SJ7" pad="2"/>
+<wire x1="29.5" y1="19" x2="31" y2="17.5" width="0.6096" layer="1"/>
+<wire x1="31" y1="17.5" x2="33" y2="17.5" width="0.6096" layer="1"/>
+<wire x1="33" y1="17.5" x2="42.078" y2="8.422" width="0.6096" layer="1"/>
+<wire x1="42.078" y1="8.422" x2="47.5" y2="8.422" width="0.6096" layer="1"/>
+<wire x1="56.5" y1="8.04" x2="56.118" y2="8.422" width="0.6096" layer="1"/>
+<wire x1="56.118" y1="8.422" x2="47.5" y2="8.422" width="0.6096" layer="1"/>
+<wire x1="29.5" y1="19" x2="25" y2="19" width="0.6096" layer="1"/>
+<wire x1="25" y1="19" x2="24.5" y2="19.5" width="0.6096" layer="1"/>
+<wire x1="24.5" y1="19.5" x2="24.5" y2="22.238" width="0.6096" layer="1"/>
+</signal>
 </signals>
